File: L1Switch/L1Switch/Net1Ports.kicad_sch (KiCad schematic)
At the start: 34 parts, among them J1 RJSNEGF8A08, T1 SM51589PEL, T2 SM51589PEL

Commit message: Connect/route 8 ports to PHY.
Parts:
- added C64, C65, C66, C67, C68, C69, C70, C71, C74, C75, C76, C77, C78, C79, C80, C81, C84, C85, C86, C87, C88, C89, C90, C91: 0.1 uF, Capacitor_SMD:C_0402_1005Metric, symbol Device:C
- added C72, C73, C82, C83, C92, C93: 1000pF, 2KV, Capacitor_SMD:C_0603_1608Metric, symbol Device:C
- added R40, R41, R42, R43, R44, R45, R46, R47, R48, R49, R50, R51, R52, R53, R54, R55, R56, R57, R58, R59, R60, R61, R62, R63, R64, R65, R66, R67, R68, R69, R70, R71, R72, R73, R74, R75: 75R0, Resistor_SMD:R_0402_1005Metric, symbol Device:R_US
- added T3, T4, T5, T6, T7, T8: SM51589PEL, L1Switch:SM51589PEL, symbol L1Switch:SM51589PEL
Connections:
- net GND: now also C64.1, C65.1, C66.1, C67.1, C68.1, C69.1, C70.1, C71.1, C74.1, C75.1, C76.1, C77.1, C78.1, C79.1, C80.1, C81.1, C84.1, C85.1, C86.1, C87.1, C88.1, C89.1, C90.1, C91.1
- net GNDPWR: now also C72.2, C73.2, C82.2, C83.2, C92.2, C93.2
- net P1.B+: now also T1.20 (TD2+); no longer T1.23 (TD1+)
- net P1.B-: now also T1.19 (TD2-); no longer T1.22 (TD1-)
- net P1.B_CMN: now also T1.21 (TCT2); no longer T1.24 (TCT1)
- net P1.C+: now also T1.17 (TD3+); no longer T1.23 (TD1+)
- net P1.C-: now also T1.16 (TD3-); no longer T1.22 (TD1-)
- net P1.C_CMN: now also T1.18 (TCT3); no longer T1.24 (TCT1)
- net P1.D+: now also T1.14 (TD4+); no longer T1.23 (TD1+)
- net P1.D-: now also T1.13 (TD4-); no longer T1.22 (TD1-)
- net P1.D_CMN: now also T1.15 (TCT4); no longer T1.24 (TCT1)
- net P2.B+: now also T2.20 (TD2+); no longer T2.23 (TD1+)
- net P2.B-: now also T2.19 (TD2-); no longer T2.22 (TD1-)
- net P2.B_CMN: now also T2.21 (TCT2); no longer T2.24 (TCT1)
- net P2.C+: now also T2.17 (TD3+); no longer T2.23 (TD1+)
- net P2.C-: now also T2.16 (TD3-); no longer T2.22 (TD1-)
- net P2.C_CMN: now also T2.18 (TCT3); no longer T2.24 (TCT1)
- net P2.D+: now also T2.14 (TD4+); no longer T2.23 (TD1+)
- net P2.D-: now also T2.13 (TD4-); no longer T2.22 (TD1-)
- net P2.D_CMN: now also T2.15 (TCT4); no longer T2.24 (TCT1)
- net TXVB_N0: now also T1.6 (MX2-); no longer T1.3 (MX1-)
- net TXVB_N1: now also T2.6 (MX2-); no longer T2.3 (MX1-)
- net TXVB_P0: now also T1.5 (MX2+); no longer T1.2 (MX1+)
- net TXVB_P1: now also T2.5 (MX2+); no longer T2.2 (MX1+)
- net TXVC_N0: now also T1.9 (MX3-); no longer T1.3 (MX1-)
- net TXVC_N1: now also T2.9 (MX3-); no longer T2.3 (MX1-)
- net TXVC_P0: now also T1.8 (MX3+); no longer T1.2 (MX1+)
- net TXVC_P1: now also T2.8 (MX3+); no longer T2.2 (MX1+)
- net TXVD_N0: now also T1.12 (MX4-); no longer T1.3 (MX1-)
- net TXVD_N1: now also T2.12 (MX4-); no longer T2.3 (MX1-)
- net TXVD_P0: now also T1.11 (MX4+); no longer T1.2 (MX1+)
- net TXVD_P1: now also T2.11 (MX4+); no longer T2.2 (MX1+)
- net at C3.2: now also T1.4 (MCT2); no longer T1.1 (MCT1)
- net at C4.2: now also T1.7 (MCT3); no longer T1.1 (MCT1)
- net at C5.2: now also T1.10 (MCT4); no longer T1.1 (MCT1)
- net at C9.2: now also T2.10 (MCT4); no longer T2.1 (MCT1)
- net at C7.2: now also T2.4 (MCT2); no longer T2.1 (MCT1)
- net at C8.2: now also T2.7 (MCT3); no longer T2.1 (MCT1)
- new net: J1.310 (3-10), R40.2
- new net: J1.312 (3-12), R41.2
- new net: J1.410 (4-10), R42.2
- new net: J1.412 (4-12), R43.2
- new net: J1.510 (5-10), R52.2
- new net: J1.512 (5-12), R53.2
- new net: J1.610 (6-10), R54.2
- new net: J1.612 (6-12), R55.2
- new net: J1.710 (7-10), R64.2
- new net: J1.712 (7-12), R65.2
- new net: J1.810 (8-10), R66.2
- new net: J1.812 (8-12), R67.2
- new net: C88.2, T8.1 (MCT1)
- new net: C82.1, R56.2, R57.2, R58.2, R59.2
- new net: C87.2, T7.10 (MCT4)
- new net: C93.1, R72.2, R73.2, R74.2, R75.2
- new net: C66.2, T3.7 (MCT3)
- new net: C90.2, T8.7 (MCT3)
- new net: C70.2, T4.7 (MCT3)
- new net: C76.2, T5.7 (MCT3)
- new net: C86.2, T7.7 (MCT3)
- new net: C75.2, T5.4 (MCT2)
- new net: C84.2, T7.1 (MCT1)
- new net: C71.2, T4.10 (MCT4)
- new net: C80.2, T6.7 (MCT3)
- new net: C79.2, T6.4 (MCT2)
- new net: C73.1, R48.2, R49.2, R50.2, R51.2
- new net: C69.2, T4.4 (MCT2)
- new net: C78.2, T6.1 (MCT1)
- new net: C85.2, T7.4 (MCT2)
- new net: C67.2, T3.10 (MCT4)
- new net: C83.1, R60.2, R61.2, R62.2, R63.2
- new net: C64.2, T3.1 (MCT1)
- new net: C81.2, T6.10 (MCT4)
- new net: C77.2, T5.10 (MCT4)
- new net: C92.1, R68.2, R69.2, R70.2, R71.2
- new net: C72.1, R44.2, R45.2, R46.2, R47.2
- new net: C89.2, T8.4 (MCT2)
- new net: C65.2, T3.4 (MCT2)
- new net: C74.2, T5.1 (MCT1)
- new net: C91.2, T8.10 (MCT4)
- new net: C68.2, T4.1 (MCT1)
- new net P3.A+: J1.31 (3-1), T3.23 (TD1+)
- new net P3.A-: J1.32 (3-2), T3.22 (TD1-)
- new net P3.A_CMN: R44.1, T3.24 (TCT1)
- new net P3.B+: J1.33 (3-3), T3.20 (TD2+)
- new net P3.B-: J1.34 (3-4), T3.19 (TD2-)
- new net P3.B_CMN: R45.1, T3.21 (TCT2)
- new net P3.C+: J1.35 (3-5), T3.17 (TD3+)
- new net P3.C-: J1.36 (3-6), T3.16 (TD3-)
- new net P3.C_CMN: R46.1, T3.18 (TCT3)
- new net P3.D+: J1.37 (3-7), T3.14 (TD4+)
- new net P3.D-: J1.38 (3-8), T3.13 (TD4-)
- new net P3.D_CMN: R47.1, T3.15 (TCT4)
- new net P3.LED0: J1.39 (3-9)
- new net P3.LED1: R40.1
- new net P3.LED2: J1.311 (3-11)
- new net P3.LED3: R41.1
- new net P4.A+: J1.41 (4-1), T4.23 (TD1+)
- new net P4.A-: J1.42 (4-2), T4.22 (TD1-)
- new net P4.A_CMN: R48.1, T4.24 (TCT1)
- new net P4.B+: J1.43 (4-3), T4.20 (TD2+)
- new net P4.B-: J1.44 (4-4), T4.19 (TD2-)
- new net P4.B_CMN: R49.1, T4.21 (TCT2)
- new net P4.C+: J1.45 (4-5), T4.17 (TD3+)
- new net P4.C-: J1.46 (4-6), T4.16 (TD3-)
- new net P4.C_CMN: R50.1, T4.18 (TCT3)
- new net P4.D+: J1.47 (4-7), T4.14 (TD4+)
- new net P4.D-: J1.48 (4-8), T4.13 (TD4-)
- new net P4.D_CMN: R51.1, T4.15 (TCT4)
- new net P4.LED0: J1.49 (4-9)
- new net P4.LED1: R42.1
- new net P4.LED2: J1.411 (4-11)
- new net P4.LED3: R43.1
- new net P5.A+: J1.51 (5-1), T5.23 (TD1+)
- new net P5.A-: J1.52 (5-2), T5.22 (TD1-)
- new net P5.A_CMN: R56.1, T5.24 (TCT1)
- new net P5.B+: J1.53 (5-3), T5.20 (TD2+)
- new net P5.B-: J1.54 (5-4), T5.19 (TD2-)
- new net P5.B_CMN: R57.1, T5.21 (TCT2)
- new net P5.C+: J1.55 (5-5), T5.17 (TD3+)
- new net P5.C-: J1.56 (5-6), T5.16 (TD3-)
- new net P5.C_CMN: R58.1, T5.18 (TCT3)
- new net P5.D+: J1.57 (5-7), T5.14 (TD4+)
- new net P5.D-: J1.58 (5-8), T5.13 (TD4-)
- new net P5.D_CMN: R59.1, T5.15 (TCT4)
- new net P5.LED0: J1.59 (5-9)
- new net P5.LED1: R52.1
- new net P5.LED2: J1.511 (5-11)
- new net P5.LED3: R53.1
- new net P6.A+: J1.61 (6-1), T6.23 (TD1+)
- new net P6.A-: J1.62 (6-2), T6.22 (TD1-)
- new net P6.A_CMN: R60.1, T6.24 (TCT1)
- new net P6.B+: J1.63 (6-3), T6.20 (TD2+)
- new net P6.B-: J1.64 (6-4), T6.19 (TD2-)
- new net P6.B_CMN: R61.1, T6.21 (TCT2)
- new net P6.C+: J1.65 (6-5), T6.17 (TD3+)
- new net P6.C-: J1.66 (6-6), T6.16 (TD3-)
- new net P6.C_CMN: R62.1, T6.18 (TCT3)
- new net P6.D+: J1.67 (6-7), T6.14 (TD4+)
- new net P6.D-: J1.68 (6-8), T6.13 (TD4-)
- new net P6.D_CMN: R63.1, T6.15 (TCT4)
- new net P6.LED0: J1.69 (6-9)
- new net P6.LED1: R54.1
- new net P6.LED2: J1.611 (6-11)
- new net P6.LED3: R55.1
- new net P7.A+: J1.71 (7-1), T7.23 (TD1+)
- new net P7.A-: J1.72 (7-2), T7.22 (TD1-)
- new net P7.A_CMN: R68.1, T7.24 (TCT1)
- new net P7.B+: J1.73 (7-3), T7.20 (TD2+)
- new net P7.B-: J1.74 (7-4), T7.19 (TD2-)
- new net P7.B_CMN: R69.1, T7.21 (TCT2)
- new net P7.C+: J1.75 (7-5), T7.17 (TD3+)
- new net P7.C-: J1.76 (7-6), T7.16 (TD3-)
- new net P7.C_CMN: R70.1, T7.18 (TCT3)
- new net P7.D+: J1.77 (7-7), T7.14 (TD4+)
- new net P7.D-: J1.78 (7-8), T7.13 (TD4-)
- new net P7.D_CMN: R71.1, T7.15 (TCT4)
- new net P7.LED0: J1.79 (7-9)
- new net P7.LED1: R64.1
- new net P7.LED2: J1.711 (7-11)
- new net P7.LED3: R65.1
- new net P8.A+: J1.81 (8-1), T8.23 (TD1+)
- new net P8.A-: J1.82 (8-2), T8.22 (TD1-)
- new net P8.A_CMN: R72.1, T8.24 (TCT1)
- new net P8.B+: J1.83 (8-3), T8.20 (TD2+)
- new net P8.B-: J1.84 (8-4), T8.19 (TD2-)
- new net P8.B_CMN: R73.1, T8.21 (TCT2)
- new net P8.C+: J1.85 (8-5), T8.17 (TD3+)
- new net P8.C-: J1.86 (8-6), T8.16 (TD3-)
- new net P8.C_CMN: R74.1, T8.18 (TCT3)
- new net P8.D+: J1.87 (8-7), T8.14 (TD4+)
- new net P8.D-: J1.88 (8-8), T8.13 (TD4-)
- new net P8.D_CMN: R75.1, T8.15 (TCT4)
- new net P8.LED0: J1.89 (8-9)
- new net P8.LED1: R66.1
- new net P8.LED2: J1.811 (8-11)
- new net P8.LED3: R67.1
- new net TXVA_N2: T3.3 (MX1-)
- new net TXVA_N3: T4.3 (MX1-)
- new net TXVA_N4: T5.3 (MX1-)
- new net TXVA_N5: T6.3 (MX1-)
- new net TXVA_N6: T7.3 (MX1-)
- new net TXVA_N7: T8.3 (MX1-)
- new net TXVA_P2: T3.2 (MX1+)
- new net TXVA_P3: T4.2 (MX1+)
- new net TXVA_P4: T5.2 (MX1+)
- new net TXVA_P5: T6.2 (MX1+)
- new net TXVA_P6: T7.2 (MX1+)
- new net TXVA_P7: T8.2 (MX1+)
- new net TXVB_N2: T3.6 (MX2-)
- new net TXVB_N3: T4.6 (MX2-)
- new net TXVB_N4: T5.6 (MX2-)
- new net TXVB_N5: T6.6 (MX2-)
- new net TXVB_N6: T7.6 (MX2-)
- new net TXVB_N7: T8.6 (MX2-)
- new net TXVB_P2: T3.5 (MX2+)
- new net TXVB_P3: T4.5 (MX2+)
- new net TXVB_P4: T5.5 (MX2+)
- new net TXVB_P5: T6.5 (MX2+)
- new net TXVB_P6: T7.5 (MX2+)
- new net TXVB_P7: T8.5 (MX2+)
- new net TXVC_N2: T3.9 (MX3-)
- new net TXVC_N3: T4.9 (MX3-)
- new net TXVC_N4: T5.9 (MX3-)
- new net TXVC_N5: T6.9 (MX3-)
- new net TXVC_N6: T7.9 (MX3-)
- new net TXVC_N7: T8.9 (MX3-)
- new net TXVC_P2: T3.8 (MX3+)
- new net TXVC_P3: T4.8 (MX3+)
- new net TXVC_P4: T5.8 (MX3+)
- new net TXVC_P5: T6.8 (MX3+)
- new net TXVC_P6: T7.8 (MX3+)
- new net TXVC_P7: T8.8 (MX3+)
- new net TXVD_N2: T3.12 (MX4-)
- new net TXVD_N3: T4.12 (MX4-)
- new net TXVD_N4: T5.12 (MX4-)
- new net TXVD_N5: T6.12 (MX4-)
- new net TXVD_N6: T7.12 (MX4-)
- new net TXVD_N7: T8.12 (MX4-)
- new net TXVD_P2: T3.11 (MX4+)
- new net TXVD_P3: T4.11 (MX4+)
- new net TXVD_P4: T5.11 (MX4+)
- new net TXVD_P5: T6.11 (MX4+)
- new net TXVD_P6: T7.11 (MX4+)
- new net TXVD_P7: T8.11 (MX4+)

Commit message: Layout replicated to Net2.
Parts:
- renumbered C2 to C166, C3 to C167, C4 to C168, C5 to C169, C6 to C170, C7 to C171, C8 to C172, C9 to C173, C1 to C174, C10 to C175, C64 to C176, C65 to C177, C66 to C178, C67 to C179, C68 to C180, C69 to C181, C70 to C182, C71 to C183, C72 to C184, C73 to C185, C74 to C186, C75 to C187, C76 to C188, C77 to C189, C78 to C190, C79 to C191, C80 to C192, C81 to C193, C82 to C194, C83 to C195, C84 to C196, C85 to C197, C86 to C198, C87 to C199, C88 to C200, C89 to C201, C90 to C202, C91 to C203, C92 to C204, C93 to C205, J1 to J5, R41 to R100, R42 to R101, R43 to R102, R44 to R103, R45 to R104, R46 to R105, R47 to R106, R48 to R107, R49 to R108, R50 to R109, R51 to R110, R52 to R111, R53 to R112, R54 to R113, R55 to R114, R56 to R115, R57 to R116, R58 to R117, R59 to R118, R60 to R119, R61 to R120, R62 to R121, R63 to R122, R64 to R123, R65 to R124, R66 to R125, R67 to R126, R68 to R127, R69 to R128, R70 to R129, R71 to R130, R72 to R131, R73 to R132, R74 to R133, R75 to R134, R36 to R87, R37 to R88, R38 to R89, R39 to R90, R4 to R91, R3 to R92, R2 to R93, R1 to R94, R5 to R95, R6 to R96, R7 to R97, R8 to R98, R40 to R99, T2 to T10, T3 to T11, T4 to T12, T5 to T13, T6 to T14, T7 to T15, T8 to T16, T1 to T9
Connections:
- net P1.B+: now also T9.23 (TD1+); no longer T9.20 (TD2+)
- net P1.B-: now also T9.22 (TD1-); no longer T9.19 (TD2-)
- net P1.B_CMN: now also T9.24 (TCT1); no longer T9.21 (TCT2)
- net P1.C+: now also T9.23 (TD1+); no longer T9.17 (TD3+)
- net P1.C-: now also T9.22 (TD1-); no longer T9.16 (TD3-)
- net P1.C_CMN: now also T9.24 (TCT1); no longer T9.18 (TCT3)
- net P1.D+: now also T9.23 (TD1+); no longer T9.14 (TD4+)
- net P1.D-: now also T9.22 (TD1-); no longer T9.13 (TD4-)
- net P1.D_CMN: now also T9.24 (TCT1); no longer T9.15 (TCT4)
- net P2.B+: now also T10.23 (TD1+); no longer T10.20 (TD2+)
- net P2.B-: now also T10.22 (TD1-); no longer T10.19 (TD2-)
- net P2.B_CMN: now also T10.24 (TCT1); no longer T10.21 (TCT2)
- net P2.C+: now also T10.23 (TD1+); no longer T10.17 (TD3+)
- net P2.C-: now also T10.22 (TD1-); no longer T10.16 (TD3-)
- net P2.C_CMN: now also T10.24 (TCT1); no longer T10.18 (TCT3)
- net P2.D+: now also T10.23 (TD1+); no longer T10.14 (TD4+)
- net P2.D-: now also T10.22 (TD1-); no longer T10.13 (TD4-)
- net P2.D_CMN: now also T10.24 (TCT1); no longer T10.15 (TCT4)
- net P3.A+: now also J5.11 (1-1); no longer J5.31 (3-1)
- net P3.A-: now also J5.12 (1-2); no longer J5.32 (3-2)
- net P3.B+: now also J5.13 (1-3), T11.23 (TD1+); no longer J5.33 (3-3), T11.20 (TD2+)
- net P3.B-: now also J5.14 (1-4), T11.22 (TD1-); no longer J5.34 (3-4), T11.19 (TD2-)
- net P3.B_CMN: now also T11.24 (TCT1); no longer T11.21 (TCT2)
- net P3.C+: now also J5.15 (1-5), T11.23 (TD1+); no longer J5.35 (3-5), T11.17 (TD3+)
- net P3.C-: now also J5.16 (1-6), T11.22 (TD1-); no longer J5.36 (3-6), T11.16 (TD3-)
- net P3.C_CMN: now also T11.24 (TCT1); no longer T11.18 (TCT3)
- net P3.D+: now also J5.17 (1-7), T11.23 (TD1+); no longer J5.37 (3-7), T11.14 (TD4+)
- net P3.D-: now also J5.18 (1-8), T11.22 (TD1-); no longer J5.38 (3-8), T11.13 (TD4-)
- net P3.D_CMN: now also T11.24 (TCT1); no longer T11.15 (TCT4)
- net P3.LED0: now also J5.19 (1-9); no longer J5.39 (3-9)
- net P3.LED2: now also J5.111 (1-11); no longer J5.311 (3-11)
- net P4.A+: now also J5.21 (2-1); no longer J5.41 (4-1)
- net P4.A-: now also J5.22 (2-2); no longer J5.42 (4-2)
- net P4.B+: now also J5.23 (2-3), T12.23 (TD1+); no longer J5.43 (4-3), T12.20 (TD2+)
- net P4.B-: now also J5.24 (2-4), T12.22 (TD1-); no longer J5.44 (4-4), T12.19 (TD2-)
- net P4.B_CMN: now also T12.24 (TCT1); no longer T12.21 (TCT2)
- net P4.C+: now also J5.25 (2-5), T12.23 (TD1+); no longer J5.45 (4-5), T12.17 (TD3+)
- net P4.C-: now also J5.26 (2-6), T12.22 (TD1-); no longer J5.46 (4-6), T12.16 (TD3-)
- net P4.C_CMN: now also T12.24 (TCT1); no longer T12.18 (TCT3)
- net P4.D+: now also J5.27 (2-7), T12.23 (TD1+); no longer J5.47 (4-7), T12.14 (TD4+)
- net P4.D-: now also J5.28 (2-8), T12.22 (TD1-); no longer J5.48 (4-8), T12.13 (TD4-)
- net P4.D_CMN: now also T12.24 (TCT1); no longer T12.15 (TCT4)
- net P4.LED0: now also J5.29 (2-9); no longer J5.49 (4-9)
- net P4.LED2: now also J5.211 (2-11); no longer J5.411 (4-11)
- net P5.A+: now also J5.11 (1-1); no longer J5.51 (5-1)
- net P5.A-: now also J5.12 (1-2); no longer J5.52 (5-2)
- net P5.B+: now also J5.13 (1-3), T13.23 (TD1+); no longer J5.53 (5-3), T13.20 (TD2+)
- net P5.B-: now also J5.14 (1-4), T13.22 (TD1-); no longer J5.54 (5-4), T13.19 (TD2-)
- net P5.B_CMN: now also T13.24 (TCT1); no longer T13.21 (TCT2)
- net P5.C+: now also J5.15 (1-5), T13.23 (TD1+); no longer J5.55 (5-5), T13.17 (TD3+)
- net P5.C-: now also J5.16 (1-6), T13.22 (TD1-); no longer J5.56 (5-6), T13.16 (TD3-)
- net P5.C_CMN: now also T13.24 (TCT1); no longer T13.18 (TCT3)
- net P5.D+: now also J5.17 (1-7), T13.23 (TD1+); no longer J5.57 (5-7), T13.14 (TD4+)
- net P5.D-: now also J5.18 (1-8), T13.22 (TD1-); no longer J5.58 (5-8), T13.13 (TD4-)
- net P5.D_CMN: now also T13.24 (TCT1); no longer T13.15 (TCT4)
- net P5.LED0: now also J5.19 (1-9); no longer J5.59 (5-9)
- net P5.LED2: now also J5.111 (1-11); no longer J5.511 (5-11)
- net P6.A+: now also J5.21 (2-1); no longer J5.61 (6-1)
- net P6.A-: now also J5.22 (2-2); no longer J5.62 (6-2)
- net P6.B+: now also J5.23 (2-3), T14.23 (TD1+); no longer J5.63 (6-3), T14.20 (TD2+)
- net P6.B-: now also J5.24 (2-4), T14.22 (TD1-); no longer J5.64 (6-4), T14.19 (TD2-)
- net P6.B_CMN: now also T14.24 (TCT1); no longer T14.21 (TCT2)
- net P6.C+: now also J5.25 (2-5), T14.23 (TD1+); no longer J5.65 (6-5), T14.17 (TD3+)
- net P6.C-: now also J5.26 (2-6), T14.22 (TD1-); no longer J5.66 (6-6), T14.16 (TD3-)
- net P6.C_CMN: now also T14.24 (TCT1); no longer T14.18 (TCT3)
- net P6.D+: now also J5.27 (2-7), T14.23 (TD1+); no longer J5.67 (6-7), T14.14 (TD4+)
- net P6.D-: now also J5.28 (2-8), T14.22 (TD1-); no longer J5.68 (6-8), T14.13 (TD4-)
- net P6.D_CMN: now also T14.24 (TCT1); no longer T14.15 (TCT4)
- net P6.LED0: now also J5.29 (2-9); no longer J5.69 (6-9)
- net P6.LED2: now also J5.211 (2-11); no longer J5.611 (6-11)
- net P7.A+: now also J5.11 (1-1); no longer J5.71 (7-1)
- net P7.A-: now also J5.12 (1-2); no longer J5.72 (7-2)
- net P7.B+: now also J5.13 (1-3), T15.23 (TD1+); no longer J5.73 (7-3), T15.20 (TD2+)
- net P7.B-: now also J5.14 (1-4), T15.22 (TD1-); no longer J5.74 (7-4), T15.19 (TD2-)
- net P7.B_CMN: now also T15.24 (TCT1); no longer T15.21 (TCT2)
- net P7.C+: now also J5.15 (1-5), T15.23 (TD1+); no longer J5.75 (7-5), T15.17 (TD3+)
- net P7.C-: now also J5.16 (1-6), T15.22 (TD1-); no longer J5.76 (7-6), T15.16 (TD3-)
- net P7.C_CMN: now also T15.24 (TCT1); no longer T15.18 (TCT3)
- net P7.D+: now also J5.17 (1-7), T15.23 (TD1+); no longer J5.77 (7-7), T15.14 (TD4+)
- net P7.D-: now also J5.18 (1-8), T15.22 (TD1-); no longer J5.78 (7-8), T15.13 (TD4-)
- net P7.D_CMN: now also T15.24 (TCT1); no longer T15.15 (TCT4)
- net P7.LED0: now also J5.19 (1-9); no longer J5.79 (7-9)
- net P7.LED2: now also J5.111 (1-11); no longer J5.711 (7-11)
- net P8.A+: now also J5.21 (2-1); no longer J5.81 (8-1)
- net P8.A-: now also J5.22 (2-2); no longer J5.82 (8-2)
- net P8.B+: now also J5.23 (2-3), T16.23 (TD1+); no longer J5.83 (8-3), T16.20 (TD2+)
- net P8.B-: now also J5.24 (2-4), T16.22 (TD1-); no longer J5.84 (8-4), T16.19 (TD2-)
- net P8.B_CMN: now also T16.24 (TCT1); no longer T16.21 (TCT2)
- net P8.C+: now also J5.25 (2-5), T16.23 (TD1+); no longer J5.85 (8-5), T16.17 (TD3+)
- net P8.C-: now also J5.26 (2-6), T16.22 (TD1-); no longer J5.86 (8-6), T16.16 (TD3-)
- net P8.C_CMN: now also T16.24 (TCT1); no longer T16.18 (TCT3)
- net P8.D+: now also J5.27 (2-7), T16.23 (TD1+); no longer J5.87 (8-7), T16.14 (TD4+)
- net P8.D-: now also J5.28 (2-8), T16.22 (TD1-); no longer J5.88 (8-8), T16.13 (TD4-)
- net P8.D_CMN: now also T16.24 (TCT1); no longer T16.15 (TCT4)
- net P8.LED0: now also J5.29 (2-9); no longer J5.89 (8-9)
- net P8.LED2: now also J5.211 (2-11); no longer J5.811 (8-11)
- net TXVB_N0: now also T9.3 (MX1-); no longer T9.6 (MX2-)
- net TXVB_N1: now also T10.3 (MX1-); no longer T10.6 (MX2-)
- net TXVB_N2: now also T11.3 (MX1-); no longer T11.6 (MX2-)
- net TXVB_N3: now also T12.3 (MX1-); no longer T12.6 (MX2-)
- net TXVB_N4: now also T13.3 (MX1-); no longer T13.6 (MX2-)
- net TXVB_N5: now also T14.3 (MX1-); no longer T14.6 (MX2-)
- net TXVB_N6: now also T15.3 (MX1-); no longer T15.6 (MX2-)
- net TXVB_N7: now also T16.3 (MX1-); no longer T16.6 (MX2-)
- net TXVB_P0: now also T9.2 (MX1+); no longer T9.5 (MX2+)
- net TXVB_P1: now also T10.2 (MX1+); no longer T10.5 (MX2+)
- net TXVB_P2: now also T11.2 (MX1+); no longer T11.5 (MX2+)
- net TXVB_P3: now also T12.2 (MX1+); no longer T12.5 (MX2+)
- net TXVB_P4: now also T13.2 (MX1+); no longer T13.5 (MX2+)
- net TXVB_P5: now also T14.2 (MX1+); no longer T14.5 (MX2+)
- net TXVB_P6: now also T15.2 (MX1+); no longer T15.5 (MX2+)
- net TXVB_P7: now also T16.2 (MX1+); no longer T16.5 (MX2+)
- net TXVC_N0: now also T9.3 (MX1-); no longer T9.9 (MX3-)
- net TXVC_N1: now also T10.3 (MX1-); no longer T10.9 (MX3-)
- net TXVC_N2: now also T11.3 (MX1-); no longer T11.9 (MX3-)
- net TXVC_N3: now also T12.3 (MX1-); no longer T12.9 (MX3-)
- net TXVC_N4: now also T13.3 (MX1-); no longer T13.9 (MX3-)
- net TXVC_N5: now also T14.3 (MX1-); no longer T14.9 (MX3-)
- net TXVC_N6: now also T15.3 (MX1-); no longer T15.9 (MX3-)
- net TXVC_N7: now also T16.3 (MX1-); no longer T16.9 (MX3-)
- net TXVC_P0: now also T9.2 (MX1+); no longer T9.8 (MX3+)
- net TXVC_P1: now also T10.2 (MX1+); no longer T10.8 (MX3+)
- net TXVC_P2: now also T11.2 (MX1+); no longer T11.8 (MX3+)
- net TXVC_P3: now also T12.2 (MX1+); no longer T12.8 (MX3+)
- net TXVC_P4: now also T13.2 (MX1+); no longer T13.8 (MX3+)
- net TXVC_P5: now also T14.2 (MX1+); no longer T14.8 (MX3+)
- net TXVC_P6: now also T15.2 (MX1+); no longer T15.8 (MX3+)
- net TXVC_P7: now also T16.2 (MX1+); no longer T16.8 (MX3+)
- net TXVD_N0: now also T9.3 (MX1-); no longer T9.12 (MX4-)
- net TXVD_N1: now also T10.3 (MX1-); no longer T10.12 (MX4-)
- net TXVD_N2: now also T11.3 (MX1-); no longer T11.12 (MX4-)
- net TXVD_N3: now also T12.3 (MX1-); no longer T12.12 (MX4-)
- net TXVD_N4: now also T13.3 (MX1-); no longer T13.12 (MX4-)
- net TXVD_N5: now also T14.3 (MX1-); no longer T14.12 (MX4-)
- net TXVD_N6: now also T15.3 (MX1-); no longer T15.12 (MX4-)
- net TXVD_N7: now also T16.3 (MX1-); no longer T16.12 (MX4-)
- net TXVD_P0: now also T9.2 (MX1+); no longer T9.11 (MX4+)
- net TXVD_P1: now also T10.2 (MX1+); no longer T10.11 (MX4+)
- net TXVD_P2: now also T11.2 (MX1+); no longer T11.11 (MX4+)
- net TXVD_P3: now also T12.2 (MX1+); no longer T12.11 (MX4+)
- net TXVD_P4: now also T13.2 (MX1+); no longer T13.11 (MX4+)
- net TXVD_P5: now also T14.2 (MX1+); no longer T14.11 (MX4+)
- net TXVD_P6: now also T15.2 (MX1+); no longer T15.11 (MX4+)
- net TXVD_P7: now also T16.2 (MX1+); no longer T16.11 (MX4+)
- net at C167.2: now also T9.1 (MCT1); no longer T9.4 (MCT2)
- net at C168.2: now also T9.1 (MCT1); no longer T9.7 (MCT3)
- net at C169.2: now also T9.1 (MCT1); no longer T9.10 (MCT4)
- net at R99.2: now also J5.110 (1-10); no longer J5.310 (3-10)
- net at R100.2: now also J5.112 (1-12); no longer J5.312 (3-12)
- net at R101.2: now also J5.210 (2-10); no longer J5.410 (4-10)
- net at R102.2: now also J5.212 (2-12); no longer J5.412 (4-12)
- net at R111.2: now also J5.110 (1-10); no longer J5.510 (5-10)
- net at R112.2: now also J5.112 (1-12); no longer J5.512 (5-12)
- net at R113.2: now also J5.210 (2-10); no longer J5.610 (6-10)
- net at R114.2: now also J5.212 (2-12); no longer J5.612 (6-12)
- net at R123.2: now also J5.110 (1-10); no longer J5.710 (7-10)
- net at R124.2: now also J5.112 (1-12); no longer J5.712 (7-12)
- net at R125.2: now also J5.210 (2-10); no longer J5.810 (8-10)
- net at R126.2: now also J5.212 (2-12); no longer J5.812 (8-12)
- net at C173.2: now also T10.1 (MCT1); no longer T10.10 (MCT4)
- net at C171.2: now also T10.1 (MCT1); no longer T10.4 (MCT2)
- net at C172.2: now also T10.1 (MCT1); no longer T10.7 (MCT3)
- net at C199.2: now also T15.1 (MCT1); no longer T15.10 (MCT4)
- net at C178.2: now also T11.1 (MCT1); no longer T11.7 (MCT3)
- net at C202.2: now also T16.1 (MCT1); no longer T16.7 (MCT3)
- net at C182.2: now also T12.1 (MCT1); no longer T12.7 (MCT3)
- net at C188.2: now also T13.1 (MCT1); no longer T13.7 (MCT3)
- net at C198.2: now also T15.1 (MCT1); no longer T15.7 (MCT3)
- net at C187.2: now also T13.1 (MCT1); no longer T13.4 (MCT2)
- net at C183.2: now also T12.1 (MCT1); no longer T12.10 (MCT4)
- net at C192.2: now also T14.1 (MCT1); no longer T14.7 (MCT3)
- net at C191.2: now also T14.1 (MCT1); no longer T14.4 (MCT2)
- net at C181.2: now also T12.1 (MCT1); no longer T12.4 (MCT2)
- net at C197.2: now also T15.1 (MCT1); no longer T15.4 (MCT2)
- net at C179.2: now also T11.1 (MCT1); no longer T11.10 (MCT4)
- net at C193.2: now also T14.1 (MCT1); no longer T14.10 (MCT4)
- net at C189.2: now also T13.1 (MCT1); no longer T13.10 (MCT4)
- net at C201.2: now also T16.1 (MCT1); no longer T16.4 (MCT2)
- net at C177.2: now also T11.1 (MCT1); no longer T11.4 (MCT2)
- net at C203.2: now also T16.1 (MCT1); no longer T16.10 (MCT4)

Commit message: Add instance 3 and 4 of the network ports.
Parts:
- renumbered C166 to C336, C167 to C337, C168 to C338, C169 to C339, C170 to C340, C171 to C341, C172 to C342, C173 to C343, C174 to C344, C175 to C345, C176 to C346, C177 to C347, C178 to C348, C179 to C349, C180 to C350, C181 to C351, C182 to C352, C183 to C353, C184 to C354, C185 to C355, C186 to C356, C187 to C357, C188 to C358, C189 to C359, C190 to C360, C191 to C361, C192 to C362, C193 to C363, C194 to C364, C195 to C365, C196 to C366, C197 to C367, C198 to C368, C199 to C369, C200 to C370, C201 to C371, C202 to C372, C203 to C373, C204 to C374, C205 to C375, J5 to J9, R87 to R208, R88 to R209, R89 to R210, R90 to R211, R91 to R212, R92 to R213, R93 to R214, R94 to R215, R95 to R216, R96 to R217, R97 to R218, R98 to R219, R99 to R220, R100 to R221, R101 to R222, R102 to R223, R103 to R224, R104 to R225, R105 to R226, R106 to R227, R107 to R228, R108 to R229, R109 to R230, R110 to R231, R111 to R232, R112 to R233, R113 to R234, R114 to R235, R115 to R236, R116 to R237, R117 to R238, R118 to R239, R119 to R240, R120 to R241, R121 to R242, R122 to R243, R123 to R244, R124 to R245, R125 to R246, R126 to R247, R127 to R248, R128 to R249, R129 to R250, R130 to R251, R131 to R252, R132 to R253, R133 to R254, R134 to R255, T9 to T25, T10 to T26, T11 to T27, T12 to T28, T13 to T29, T14 to T30, T15 to T31, T16 to T32
