File: L1Switch/L1Switch/Net1Ports.kicad_sch (KiCad schematic)
At the start: 124 parts, among them J9 RJSNEGF8A08, T25 SM51589PEL, T26 SM51589PEL, T27 SM51589PEL, T28 SM51589PEL, T29 SM51589PEL, T30 SM51589PEL, T31 SM51589PEL, T32 SM51589PEL

Commit message: Swap fan connector orientation. Add PU/PD for JTAG pins.
Parts:
- renumbered C344 to C1, C345 to C10, C336 to C2, C337 to C3, C338 to C4, C339 to C5, C340 to C6, C346 to C64, C347 to C65, C348 to C66, C349 to C67, C350 to C68, C351 to C69, C341 to C7, C352 to C70, C353 to C71, C354 to C72, C355 to C73, C356 to C74, C357 to C75, C358 to C76, C359 to C77, C360 to C78, C361 to C79, C342 to C8, C362 to C80, C363 to C81, C364 to C82, C365 to C83, C366 to C84, C367 to C85, C368 to C86, C369 to C87, C370 to C88, C371 to C89, C343 to C9, C372 to C90, C373 to C91, C374 to C92, C375 to C93, J9 to J1, R215 to R1, R214 to R2, R213 to R3, R208 to R36, R209 to R37, R210 to R38, R211 to R39, R212 to R4, R220 to R40, R221 to R41, R222 to R42, R223 to R43, R224 to R44, R225 to R45, R226 to R46, R227 to R47, R228 to R48, R229 to R49, R216 to R5, R230 to R50, R231 to R51, R232 to R52, R233 to R53, R234 to R54, R235 to R55, R236 to R56, R237 to R57, R238 to R58, R239 to R59, R217 to R6, R240 to R60, R241 to R61, R242 to R62, R243 to R63, R244 to R64, R245 to R65, R246 to R66, R247 to R67, R248 to R68, R249 to R69, R218 to R7, R250 to R70, R251 to R71, R252 to R72, R253 to R73, R254 to R74, R255 to R75, R219 to R8, T25 to T1, T26 to T2, T27 to T3, T28 to T4, T29 to T5, T30 to T6, T31 to T7, T32 to T8

Commit message: Update RJ45 pinout on schematic and partial layout update.
Connections:
- net P1.B-: now also J1.16 (1-6); no longer J1.14 (1-4)
- net P1.C+: now also J1.14 (1-4); no longer J1.15 (1-5)
- net P1.C-: now also J1.15 (1-5); no longer J1.16 (1-6)
- net P2.B-: now also J1.26 (2-6); no longer J1.24 (2-4)
- net P2.C+: now also J1.24 (2-4); no longer J1.25 (2-5)
- net P2.C-: now also J1.25 (2-5); no longer J1.26 (2-6)
- net P3.B-: now also J1.16 (1-6); no longer J1.14 (1-4)
- net P3.C+: now also J1.14 (1-4); no longer J1.15 (1-5)
- net P3.C-: now also J1.15 (1-5); no longer J1.16 (1-6)
- net P4.B-: now also J1.26 (2-6); no longer J1.24 (2-4)
- net P4.C+: now also J1.24 (2-4); no longer J1.25 (2-5)
- net P4.C-: now also J1.25 (2-5); no longer J1.26 (2-6)
- net P5.B-: now also J1.16 (1-6); no longer J1.14 (1-4)
- net P5.C+: now also J1.14 (1-4); no longer J1.15 (1-5)
- net P5.C-: now also J1.15 (1-5); no longer J1.16 (1-6)
- net P6.B-: now also J1.26 (2-6); no longer J1.24 (2-4)
- net P6.C+: now also J1.24 (2-4); no longer J1.25 (2-5)
- net P6.C-: now also J1.25 (2-5); no longer J1.26 (2-6)
- net P7.B-: now also J1.16 (1-6); no longer J1.14 (1-4)
- net P7.C+: now also J1.14 (1-4); no longer J1.15 (1-5)
- net P7.C-: now also J1.15 (1-5); no longer J1.16 (1-6)
- net P8.B-: now also J1.26 (2-6); no longer J1.24 (2-4)
- net P8.C+: now also J1.24 (2-4); no longer J1.25 (2-5)
- net P8.C-: now also J1.25 (2-5); no longer J1.26 (2-6)

Commit message: Update voltage monitoring.
Parts:
- renumbered C2 to C336, C3 to C337, C4 to C338, C5 to C339, C6 to C340, C7 to C341, C8 to C342, C9 to C343, C1 to C344, C10 to C345, C64 to C346, C65 to C347, C66 to C348, C67 to C349, C68 to C350, C69 to C351, C70 to C352, C71 to C353, C72 to C354, C73 to C355, C74 to C356, C75 to C357, C76 to C358, C77 to C359, C78 to C360, C79 to C361, C80 to C362, C81 to C363, C82 to C364, C83 to C365, C84 to C366, C85 to C367, C86 to C368, C87 to C369, C88 to C370, C89 to C371, C90 to C372, C91 to C373, C92 to C374, C93 to C375, J1 to J9, R36 to R208, R37 to R209, R38 to R210, R39 to R211, R4 to R212, R3 to R213, R2 to R214, R1 to R215, R5 to R216, R6 to R217, R7 to R218, R8 to R219, R40 to R220, R41 to R221, R42 to R222, R43 to R223, R44 to R224, R45 to R225, R46 to R226, R47 to R227, R48 to R228, R49 to R229, R50 to R230, R51 to R231, R52 to R232, R53 to R233, R54 to R234, R55 to R235, R56 to R236, R57 to R237, R58 to R238, R59 to R239, R60 to R240, R61 to R241, R62 to R242, R63 to R243, R64 to R244, R65 to R245, R66 to R246, R67 to R247, R68 to R248, R69 to R249, R70 to R250, R71 to R251, R72 to R252, R73 to R253, R74 to R254, R75 to R255, T1 to T25, T2 to T26, T3 to T27, T4 to T28, T5 to T29, T6 to T30, T7 to T31, T8 to T32
