File: L1Switch/L1Switch/Power.kicad_sch (KiCad schematic)
At the start: 60 parts, among them J3 Barrel_Jack, U3 TPS548A20RVE, U4 TPS565208, U5 TPS565208, U6 TPS565208

Commit message: Most signals routed.
Connections:
- no-connect marks 0 -> 1
Changed lines of the file:
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@@
 (kicad_sch (version 20200608) (host eeschema "5.99.0-unknown-1973153~101~ubuntu20.04.1")
-  (page 1 12)
+  (page 12 12)
   (paper "B")
   (junction (at 26.67 80.01))
@@
   (junction (at 396.24 143.51))
   (junction (at 396.24 182.88))
+  (no_connect (at 345.44 55.88))
   (wire (pts (xy 20.32 48.26) (xy 29.21 48.26))
     (stroke (width 0) (type solid) (color 0 0 0 0))
